Commit message: feat: 借鉴 OOMWOO 架构（Safety + 模块化 URDF）
借鉴 https://github.com/makerspet/oomwoo 的 3 个架构思想：

1. Safety 跑在 MCU（v3 firmware）：
   - ESP32 firmware v3：safety.h/cc + main_v3.cpp
   - 急停按钮 + 4 个 bumper + 低电量监测
   - 不依赖 ROS2，ROS2 挂了也能急停
   - 双任务：50Hz 控制 + 1Hz safety log

2. 模块化 URDF（借鉴 oomwoo-one）：
   - urdf/xacro/params.xacro 集中参数
   - urdf/xacro/inertial.xacro 惯性宏
   - urdf/xacro/materials.xacro 材质
   - urdf/xacro/wheels.xacro 底盘/轮子宏
   - urdf/xacro/sensors.xacro 传感器宏
   - urdf/slam_robot.urdf.xacro 主 URDF（5 行 macro 调用）
   - 7 link + 6 joint

3. ARCHITECTURE.md（借鉴 Oomwoo）：
   - 设计原则：CPU+MCU 分离 / Safety 不依赖 ROS2 / 模块化
   - 系统框图
   - 模块清单
   - 数据流图
   - 与 Oomwoo 的差异化对比

Made-with: Proma

File: urdf/slam_robot.urdf.xacro (robot description, xacro)
@@ -1,225 +1,31 @@
 <?xml version="1.0"?>
-<robot xmlns:xacro="http://www.ros.org/wiki/xacro" name="slam_robot">
-  <!-- ====================================================== -->
-  <!-- 常量 -->
-  <!-- ====================================================== -->
-  <xacro:property name="base_length" value="0.50"/>
-  <xacro:property name="base_width" value="0.35"/>
-  <xacro:property name="base_height" value="0.12"/>
-  <xacro:property name="base_mass" value="3.0"/>
-  <xacro:property name="wheel_radius" value="0.06"/>
-  <xacro:property name="wheel_width" value="0.04"/>
-  <xacro:property name="wheel_mass" value="0.2"/>
-  <xacro:property name="laser_height" value="0.30"/>  <!-- 雷达离地 0.30 m -->
-  <xacro:property name="imu_height" value="0.10"/>
-  <xacro:property name="PI" value="3.14159265359"/>
-  <!-- ====================================================== -->
-  <!-- 底盘 base_link -->
-  <!-- ====================================================== -->
-  <link name="base_link">
-    <visual>
-      <origin xyz="0 0 ${base_height/2}" rpy="0 0 0"/>
-      <geometry>
-        <box size="${base_length} ${base_width} ${base_height}"/>
-      </geometry>
-      <material name="gray">
-        <color rgba="0.5 0.5 0.5 1"/>
-      </material>
-    </visual>
-    <collision>
-      <origin xyz="0 0 ${base_height/2}" rpy="0 0 0"/>
-      <geometry>
-        <box size="${base_length} ${base_width} ${base_height}"/>
-      </geometry>
-    </collision>
-    <inertial>
-      <origin xyz="0 0 ${base_height/2}" rpy="0 0 0"/>
-      <mass value="${base_mass}"/>
-      <inertia ixx="0.1" ixy="0" ixz="0" iyy="0.2" iyz="0" izz="0.2"/>
-    </inertial>
-  </link>
-  <!-- ====================================================== -->
-  <!-- 左驱动轮 wheel_left_link -->
-  <!-- ====================================================== -->
-  <link name="wheel_left_link">
-    <visual>
-      <origin xyz="0 0 0" rpy="0 0 0"/>
-      <geometry>
-        <cylinder radius="${wheel_radius}" length="${wheel_width}"/>
-      </geometry>
-      <material name="black">
-        <color rgba="0 0 0 1"/>
-      </material>
-    </visual>
-    <collision>
-      <origin xyz="0 0 0" rpy="0 0 0"/>
-      <geometry>
-        <cylinder radius="${wheel_radius}" length="${wheel_width}"/>
-      </geometry>
-    </collision>
-    <inertial>
-      <origin xyz="0 0 0" rpy="0 0 0"/>
-      <mass value="${wheel_mass}"/>
-      <inertia ixx="0.01" ixy="0" ixz="0" iyy="0.01" iyz="0" izz="0.005"/>
-    </inertial>
-  </link>
-  <joint name="wheel_left_joint" type="continuous">
-    <parent link="base_link"/>
-    <child link="wheel_left_link"/>
-    <origin xyz="0 ${base_width/2 + wheel_width/2} 0" rpy="-${PI/2} 0 0"/>
-    <axis xyz="0 0 1"/>
-    <dynamics damping="0.1" friction="0.1"/>
-  </joint>
-  <!-- ====================================================== -->
-  <!-- 右驱动轮 wheel_right_link -->
-  <!-- ====================================================== -->
-  <link name="wheel_right_link">
-    <visual>
-      <origin xyz="0 0 0" rpy="0 0 0"/>
-      <geometry>
-        <cylinder radius="${wheel_radius}" length="${wheel_width}"/>
-      </geometry>
-      <material name="black">
-        <color rgba="0 0 0 1"/>
-      </material>
-    </visual>
-    <collision>
-      <origin xyz="0 0 0" rpy="0 0 0"/>
-      <geometry>
-        <cylinder radius="${wheel_radius}" length="${wheel_width}"/>
-      </geometry>
-    </collision>
-    <inertial>
-      <origin xyz="0 0 0" rpy="0 0 0"/>
-      <mass value="${wheel_mass}"/>
-      <inertia ixx="0.01" ixy="0" ixz="0" iyy="0.01" iyz="0" izz="0.005"/>
-    </inertial>
-  </link>
-  <joint name="wheel_right_joint" type="continuous">
-    <parent link="base_link"/>
-    <child link="wheel_right_link"/>
-    <origin xyz="0 ${-(base_width/2 + wheel_width/2)} 0" rpy="-${PI/2} 0 0"/>
-    <axis xyz="0 0 1"/>
-    <dynamics damping="0.1" friction="0.1"/>
-  </joint>
-  <!-- ====================================================== -->
-  <!-- 前万向轮 caster_front_link（固定 joint，无驱动） -->
-  <!-- ====================================================== -->
-  <link name="caster_front_link">
-    <visual>
-      <origin xyz="0 0 0" rpy="0 0 0"/>
-      <geometry>
-        <sphere radius="0.025"/>
-      </geometry>
-      <material name="black">
-        <color rgba="0 0 0 1"/>
-      </material>
-    </visual>
-    <collision>
-      <origin xyz="0 0 0" rpy="0 0 0"/>
-      <geometry>
-        <sphere radius="0.025"/>
-      </geometry>
-    </collision>
-    <inertial>
-      <origin xyz="0 0 0" rpy="0 0 0"/>
-      <mass value="0.05"/>
-      <inertia ixx="0.001" ixy="0" ixz="0" iyy="0.001" iyz="0" izz="0.001"/>
-    </inertial>
-  </link>
-  <joint name="caster_front_joint" type="fixed">
-    <parent link="base_link"/>
-    <child link="caster_front_link"/>
-    <origin xyz="${base_length/2 - 0.05} 0 0" rpy="0 0 0"/>
-  </joint>
-  <!-- ====================================================== -->
-  <!-- 后万向轮 caster_back_link（可选） -->
-  <!-- ====================================================== -->
-  <link name="caster_back_link">
-    <visual>
-      <origin xyz="0 0 0" rpy="0 0 0"/>
-      <geometry>
-        <sphere radius="0.025"/>
-      </geometry>
-      <material name="black">
-        <color rgba="0 0 0 1"/>
-      </material>
-    </visual>
-    <collision>
-      <origin xyz="0 0 0" rpy="0 0 0"/>
-      <geometry>
-        <sphere radius="0.025"/>
-      </geometry>
-    </collision>
-    <inertial>
-      <origin xyz="0 0 0" rpy="0 0 0"/>
-      <mass value="0.05"/>
-      <inertia ixx="0.001" ixy="0" ixz="0" iyy="0.001" iyz="0" izz="0.001"/>
-    </inertial>
-  </link>
-  <joint name="caster_back_joint" type="fixed">
-    <parent link="base_link"/>
-    <child link="caster_back_link"/>
-    <origin xyz="${-(base_length/2 - 0.05)} 0 0" rpy="0 0 0"/>
-  </joint>
-  <!-- ====================================================== -->
-  <!-- 激光雷达 laser_frame -->
-  <!-- ====================================================== -->
-  <link name="laser_frame">
-    <visual>
-      <origin xyz="0 0 0" rpy="0 0 0"/>
-      <geometry>
-        <cylinder radius="0.04" length="0.04"/>
-      </geometry>
-      <material name="green">
-        <color rgba="0 1 0 1"/>
-      </material>
-    </visual>
-    <collision>
-      <origin xyz="0 0 0" rpy="0 0 0"/>
-      <geometry>
-        <cylinder radius="0.04" length="0.04"/>
-      </geometry>
-    </collision>
-    <inertial>
-      <origin xyz="0 0 0" rpy="0 0 0"/>
-      <mass value="0.1"/>
-      <inertia ixx="0.001" ixy="0" ixz="0" iyy="0.001" iyz="0" izz="0.001"/>
-    </inertial>
-  </link>
-  <joint name="laser_joint" type="fixed">
-    <parent link="base_link"/>
-    <child link="laser_frame"/>
-    <origin xyz="0 0 ${laser_height}" rpy="0 0 0"/>
-  </joint>
-  <!-- ====================================================== -->
-  <!-- IMU imu_link -->
-  <!-- ====================================================== -->
-  <link name="imu_link">
-    <visual>
-      <origin xyz="0 0 0" rpy="0 0 0"/>
-      <geometry>
-        <box size="0.02 0.02 0.005"/>
-      </geometry>
-      <material name="blue">
-        <color rgba="0 0 1 1"/>
-      </material>
-    </visual>
-    <collision>
-      <origin xyz="0 0 0" rpy="0 0 0"/>
-      <geometry>
-        <box size="0.02 0.02 0.005"/>
-      </geometry>
-    </collision>
-    <inertial>
-      <origin xyz="0 0 0" rpy="0 0 0"/>
-      <mass value="0.01"/>
-      <inertia ixx="0.0001" ixy="0" ixz="0" iyy="0.0001" iyz="0" izz="0.0001"/>
-    </inertial>
-  </link>
-  <joint name="imu_joint" type="fixed">
-    <parent link="base_link"/>
-    <child link="imu_link"/>
-    <origin xyz="0 0 ${imu_height}" rpy="0 0 0"/>
-  </joint>
+<!--
+  SLAM 机器人 URDF（借鉴 oomwoo-one 模块化设计）
+  - params.xacro：参数
+  - inertial.xacro：惯性宏
+  - materials.xacro：材质
+  - wheels.xacro：底盘 / 轮子宏
+  - sensors.xacro：传感器宏
+-->
+<robot xmlns:xacro="http://ros.org/wiki/xacro" name="slam_robot">
+  <!-- 加载子模块 -->
+  <xacro:include filename="$(find indoor_slam_67m)/urdf/xacro/params.xacro"/>
+  <xacro:include filename="$(find indoor_slam_67m)/urdf/xacro/materials.xacro"/>
+  <xacro:include filename="$(find indoor_slam_67m)/urdf/xacro/inertial.xacro"/>
+  <xacro:include filename="$(find indoor_slam_67m)/urdf/xacro/wheels.xacro"/>
+  <xacro:include filename="$(find indoor_slam_67m)/urdf/xacro/sensors.xacro"/>
+  <!-- 底盘主体 -->
+  <xacro:base_body base_length="${base_length}"
+                   base_width="${base_width}"
+                   base_height="${base_height}"
+                   base_mass="${base_mass}"/>
+  <!-- 驱动轮 -->
+  <xacro:drive_wheel side="left"  wheel_radius="${wheel_radius}" wheel_mass="${wheel_mass}" y_position="${base_width/2 + base_width/8}"/>
+  <xacro:drive_wheel side="right" wheel_radius="${wheel_radius}" wheel_mass="${wheel_mass}" y_position="${-(base_width/2 + base_width/8)}"/>
+  <!-- 万向轮（前 + 后） -->
+  <xacro:caster_wheel position="front" caster_radius="${caster_radius}" x_position="${base_length/2 - 0.05}"/>
+  <xacro:caster_wheel position="back"  caster_radius="${caster_radius}" x_position="${-(base_length/2 - 0.05)}"/>
+  <!-- 传感器 -->
+  <xacro:laser_sensor x="0" y="0" z="${laser_height}"/>
+  <xacro:imu_sensor   x="0" y="0" z="${imu_height}"/>
 </robot>
